Commit message: refactor(std): 扁平化描述包到仓库根目录并统一 std 命名
将 ROS 2 包从 src/standrad/ 扁平化到仓库根目录, 包名统一为 bw_std_description, 配套重命名 config、rviz、scripts、urdf 与 CMake 元数据。

运行时模型改名为 std_auto, 六个显示模型统一为 std_v1 至 std_v6, 生成脚本改为以 std_auto.urdf 为源模型输出显示模型。

启动参数 variant 改为 robot_model, 支持列表加入 std_auto, 非法取值直接报错并列出可选值, Gazebo 实体名默认改为 std_robot。

URDF 与 std_source.csv 中的资源引用统一为 package://bw_std_description/, Gazebo 启动时把该前缀替换为本地绝对路径。

117 个 STL 与 std.rviz、joint_names_std.yaml 仅移动或改名, 文件内容未变。

README 更新为新目录结构与新参数名, 补充 model、rviz_config、entity_name 等可选启动参数说明。

旧包名 standard 与旧参数 variant 不再支持。

File: urdf/std_auto.urdf (robot description, URDF)
Before this commit: robot standard, 27 links, 26 joints
Links:
- link A_left_Degree1_link: geometry collision mesh filename=package://bw_std_description/meshes/A_left_Degree1_link.STL; visual mesh filename=package://bw_std_description/meshes/A_left_Degree1_link.STL
- link A_left_Degree2_link: geometry collision mesh filename=package://bw_std_description/meshes/A_left_Degree2_link.STL; visual mesh filename=package://bw_std_description/meshes/A_left_Degree2_link.STL
- link A_left_Degree3_link: geometry collision mesh filename=package://bw_std_description/meshes/A_left_Degree3_link.STL; visual mesh filename=package://bw_std_description/meshes/A_left_Degree3_link.STL
- link A_left_Degree4_link: geometry collision mesh filename=package://bw_std_description/meshes/A_left_Degree4_link.STL; visual mesh filename=package://bw_std_description/meshes/A_left_Degree4_link.STL
- link A_left_Degree5_link: geometry collision mesh filename=package://bw_std_description/meshes/A_left_Degree5_link.STL; visual mesh filename=package://bw_std_description/meshes/A_left_Degree5_link.STL
- link A_left_Degree6_link: geometry collision mesh filename=package://bw_std_description/meshes/A_left_Degree6_link.STL; visual mesh filename=package://bw_std_description/meshes/A_left_Degree6_link.STL
- link A_left_Degree7_link: geometry collision mesh filename=package://bw_std_description/meshes/A_left_Degree7_link.STL; visual mesh filename=package://bw_std_description/meshes/A_left_Degree7_link.STL
- link A_left_Degree8_link: geometry collision mesh filename=package://bw_std_description/meshes/A_left_Degree8_link.STL; visual mesh filename=package://bw_std_description/meshes/A_left_Degree8_link.STL
- link A_left_Degree9_link: geometry collision mesh filename=package://bw_std_description/meshes/A_left_Degree9_link.STL; visual mesh filename=package://bw_std_description/meshes/A_left_Degree9_link.STL
- link A_right_Degree1_link: geometry collision mesh filename=package://bw_std_description/meshes/A_right_Degree1_link.STL; visual mesh filename=package://bw_std_description/meshes/A_right_Degree1_link.STL
- link A_right_Degree2_link: geometry collision mesh filename=package://bw_std_description/meshes/A_right_Degree2_link.STL; visual mesh filename=package://bw_std_description/meshes/A_right_Degree2_link.STL
- link A_right_Degree3_link: geometry collision mesh filename=package://bw_std_description/meshes/A_right_Degree3_link.STL; visual mesh filename=package://bw_std_description/meshes/A_right_Degree3_link.STL
- link A_right_Degree4_link: geometry collision mesh filename=package://bw_std_description/meshes/A_right_Degree4_link.STL; visual mesh filename=package://bw_std_description/meshes/A_right_Degree4_link.STL
- link A_right_Degree5_link: geometry collision mesh filename=package://bw_std_description/meshes/A_right_Degree5_link.STL; visual mesh filename=package://bw_std_description/meshes/A_right_Degree5_link.STL
- link A_right_Degree6_link: geometry collision mesh filename=package://bw_std_description/meshes/A_right_Degree6_link.STL; visual mesh filename=package://bw_std_description/meshes/A_right_Degree6_link.STL
- link A_right_Degree7_link: geometry collision mesh filename=package://bw_std_description/meshes/A_right_Degree7_link.STL; visual mesh filename=package://bw_std_description/meshes/A_right_Degree7_link.STL
- link A_right_Degree8_link: geometry collision mesh filename=package://bw_std_description/meshes/A_right_Degree8_link.STL; visual mesh filename=package://bw_std_description/meshes/A_right_Degree8_link.STL
- link A_right_Degree9_link: geometry collision mesh filename=package://bw_std_description/meshes/A_right_Degree9_link.STL; visual mesh filename=package://bw_std_description/meshes/A_right_Degree9_link.STL
- link C_Link: geometry collision mesh filename=package://bw_std_description/meshes/C_Link.STL; visual mesh filename=package://bw_std_description/meshes/C_Link.STL
- link D_behind_Link: geometry collision mesh filename=package://bw_std_description/meshes/D_behind_Link.STL; visual mesh filename=package://bw_std_description/meshes/D_behind_Link.STL
- link D_left_Link: geometry collision mesh filename=package://bw_std_description/meshes/D_left_Link.STL; visual mesh filename=package://bw_std_description/meshes/D_left_Link.STL
- link D_right_Link: geometry collision mesh filename=package://bw_std_description/meshes/D_right_Link.STL; visual mesh filename=package://bw_std_description/meshes/D_right_Link.STL
- link H_Degree1_Link: geometry collision mesh filename=package://bw_std_description/meshes/H_Degree1_Link.STL; visual mesh filename=package://bw_std_description/meshes/H_Degree1_Link.STL
- link H_Degree2_link: geometry collision mesh filename=package://bw_std_description/meshes/H_Degree2_link.STL; visual mesh filename=package://bw_std_description/meshes/H_Degree2_link.STL
- link H_Degree3_link: geometry collision mesh filename=package://bw_std_description/meshes/H_Degree3_link.STL; visual mesh filename=package://bw_std_description/meshes/H_Degree3_link.STL
- link base_link: geometry collision mesh filename=package://bw_std_description/meshes/base_link.STL; visual mesh filename=package://bw_std_description/meshes/base_link.STL

File: urdf/std_v1.urdf (robot description, URDF)
Before this commit: robot standard_v2, 22 links, 21 joints
Links:
- removed link chest_top_cap
- removed link linear_slide_link
- added link D_behind_Link, mass 0.462675307874263; collision mesh filename=package://bw_std_description/meshes/v1/D_behind_Link.STL; visual mesh filename=package://bw_std_description/meshes/v1/D_behind_Link.STL
- added link D_left_Link, mass 0.462675291076093; collision mesh filename=package://bw_std_description/meshes/v1/D_left_Link.STL; visual mesh filename=package://bw_std_description/meshes/v1/D_left_Link.STL
- added link D_right_Link, mass 0.462675301767314; collision mesh filename=package://bw_std_description/meshes/v1/D_right_Link.STL; visual mesh filename=package://bw_std_description/meshes/v1/D_right_Link.STL
- added link H_Degree1_Link, mass 0.448403215424371; collision mesh filename=package://bw_std_description/meshes/v1/H_Degree1_Link.STL; visual mesh filename=package://bw_std_description/meshes/v1/H_Degree1_Link.STL
- added link H_Degree2_link, mass 0.391963477171488; collision mesh filename=package://bw_std_description/meshes/v1/H_Degree2_link.STL; visual mesh filename=package://bw_std_description/meshes/v1/H_Degree2_link.STL
- added link H_Degree3_link, mass 17.1573718140124; collision mesh filename=package://bw_std_description/meshes/v1/H_Degree3_link.STL; visual mesh filename=package://bw_std_description/meshes/v1/H_Degree3_link.STL
- added link base_link, mass 13.9911595310973; collision mesh filename=package://bw_std_description/meshes/v1/base_link.STL; visual mesh filename=package://bw_std_description/meshes/v1/base_link.STL
- link A_left_Degree1_link: geometry collision mesh filename=package://bw_std_description/meshes/v1/A_left_Degree1_link.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; visual mesh filename=package://bw_std_description/meshes/v1/A_left_Degree1_link.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
- link A_left_Degree2_link: geometry collision mesh filename=package://bw_std_description/meshes/v1/A_left_Degree2_link.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; visual mesh filename=package://bw_std_description/meshes/v1/A_left_Degree2_link.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
- link A_left_Degree3_link: geometry collision mesh filename=package://bw_std_description/meshes/v1/A_left_Degree3_link.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; visual mesh filename=package://bw_std_description/meshes/v1/A_left_Degree3_link.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
- link A_left_Degree4_link: geometry collision mesh filename=package://bw_std_description/meshes/v1/A_left_Degree4_link.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; visual mesh filename=package://bw_std_description/meshes/v1/A_left_Degree4_link.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
- link A_left_Degree5_link: geometry collision mesh filename=package://bw_std_description/meshes/v1/A_left_Degree5_link.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; visual mesh filename=package://bw_std_description/meshes/v1/A_left_Degree5_link.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
- link A_left_Degree6_link: geometry collision mesh filename=package://bw_std_description/meshes/v1/A_left_Degree6_link.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; visual mesh filename=package://bw_std_description/meshes/v1/A_left_Degree6_link.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
- link A_left_Degree7_link: geometry collision mesh filename=package://bw_std_description/meshes/v1/A_left_Degree7_link.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; visual mesh filename=package://bw_std_description/meshes/v1/A_left_Degree7_link.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
- link A_left_Degree8_link: geometry collision mesh filename=package://bw_std_description/meshes/v1/A_left_Degree8_link.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; visual mesh filename=package://bw_std_description/meshes/v1/A_left_Degree8_link.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
- link A_left_Degree9_link: geometry collision mesh filename=package://bw_std_description/meshes/v1/A_left_Degree9_link.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; visual mesh filename=package://bw_std_description/meshes/v1/A_left_Degree9_link.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
- link A_right_Degree1_link: geometry collision mesh filename=package://bw_std_description/meshes/v1/A_right_Degree1_link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; visual mesh filename=package://bw_std_description/meshes/v1/A_right_Degree1_link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
- link A_right_Degree2_link: geometry collision mesh filename=package://bw_std_description/meshes/v1/A_right_Degree2_link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; visual mesh filename=package://bw_std_description/meshes/v1/A_right_Degree2_link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
- link A_right_Degree3_link: geometry collision mesh filename=package://bw_std_description/meshes/v1/A_right_Degree3_link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; visual mesh filename=package://bw_std_description/meshes/v1/A_right_Degree3_link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
- link A_right_Degree4_link: geometry collision mesh filename=package://bw_std_description/meshes/v1/A_right_Degree4_link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; visual mesh filename=package://bw_std_description/meshes/v1/A_right_Degree4_link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
- link A_right_Degree5_link: geometry collision mesh filename=package://bw_std_description/meshes/v1/A_right_Degree5_link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; visual mesh filename=package://bw_std_description/meshes/v1/A_right_Degree5_link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
- link A_right_Degree6_link: geometry collision mesh filename=package://bw_std_description/meshes/v1/A_right_Degree6_link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; visual mesh filename=package://bw_std_description/meshes/v1/A_right_Degree6_link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
- link A_right_Degree7_link: geometry collision mesh filename=package://bw_std_description/meshes/v1/A_right_Degree7_link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; visual mesh filename=package://bw_std_description/meshes/v1/A_right_Degree7_link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
- link A_right_Degree8_link: geometry collision mesh filename=package://bw_std_description/meshes/v1/A_right_Degree8_link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; visual mesh filename=package://bw_std_description/meshes/v1/A_right_Degree8_link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
- link A_right_Degree9_link: geometry collision mesh filename=package://bw_std_description/meshes/v1/A_right_Degree9_link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; visual mesh filename=package://bw_std_description/meshes/v1/A_right_Degree9_link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
- link C_Link: geometry collision mesh filename=package://bw_std_description/meshes/v1/C_Link.STL; visual mesh filename=package://bw_std_description/meshes/v1/C_Link.STL
Joints:
- removed joint chest_top_cap_joint
- removed joint linear_slide_joint
- added joint D_behind_joint: type continuous, parent base_link, child D_behind_Link, origin xyz=-0.248002748938563 0 0.0394999999999985 rpy=0 0 3.14159248134972, axis -1 0 0, limit lower=0 upper=0 effort=0 velocity=0
- added joint D_left_joint: type continuous, parent base_link, child D_left_Link, origin xyz=0.124001411462432 0.214776659431165 0.0394999999999984 rpy=3.14159265358979 0 -2.09439527463327, axis -1 0 0, limit lower=0 upper=0 effort=0 velocity=0
- added joint D_right_joint: type continuous, parent base_link, child D_right_Link, origin xyz=0.124001337476132 -0.214776702147174 0.0394999999999984 rpy=3.14159265358979 0 -1.04719772343667, axis -1 0 0, limit lower=0 upper=0 effort=0 velocity=0
- added joint H_Degree1_joint: type revolute, parent C_Link, child H_Degree1_Link, origin xyz=0.0966216027047007 0 0.0795707701001659 rpy=0 0 0, axis 0 0 1, limit lower=-2.0944 upper=2.0944 effort=0 velocity=0
- added joint H_Degree2_joint: type revolute, parent H_Degree1_Link, child H_Degree2_link, origin xyz=-0.07435450768229898 1.281731919551012e-08 0.1197410391411445 rpy=0 0 0, axis 1 0 0, limit lower=-0.6981 upper=0.6981 effort=0 velocity=0
- added joint H_Degree3_joint: type revolute, parent H_Degree2_link, child H_Degree3_link, origin xyz=0.09961620127967459 0.06850022646523188 -4.955647739572536e-05 rpy=0 0 0, axis 0 1 0, limit lower=-0.7854 upper=0.7854 effort=0 velocity=0
- added joint base_footprint_to_base_link: type fixed, parent base_footprint, child base_link, origin xyz=0 0 0 rpy=0 0 0
- joint C_joint: parent base_footprint -> base_link

File: urdf/std_v2.urdf (robot description, URDF)
Before this commit: robot standard_v1, 27 links, 26 joints
Links:
- removed link D_behind_Link
- removed link D_left_Link
- removed link D_right_Link
- removed link H_Degree1_Link
- removed link H_Degree2_link
- removed link H_Degree3_link
- removed link base_link
- added link chest_top_cap; collision mesh filename=package://bw_std_description/meshes/v2/chest_top_cap.STL; visual mesh filename=package://bw_std_description/meshes/v2/chest_top_cap.STL
- added link linear_slide_link; collision mesh filename=package://bw_std_description/meshes/v2/linear_slide_v2.STL; visual mesh filename=package://bw_std_description/meshes/v2/linear_slide_v2.STL
- link A_left_Degree1_link: geometry collision mesh filename=package://bw_std_description/meshes/v2/A_left_Degree1_link.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; visual mesh filename=package://bw_std_description/meshes/v2/A_left_Degree1_link.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
- link A_left_Degree2_link: geometry collision mesh filename=package://bw_std_description/meshes/v2/A_left_Degree2_link.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; visual mesh filename=package://bw_std_description/meshes/v2/A_left_Degree2_link.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
- link A_left_Degree3_link: geometry collision mesh filename=package://bw_std_description/meshes/v2/A_left_Degree3_link.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; visual mesh filename=package://bw_std_description/meshes/v2/A_left_Degree3_link.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
- link A_left_Degree4_link: geometry collision mesh filename=package://bw_std_description/meshes/v2/A_left_Degree4_link.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; visual mesh filename=package://bw_std_description/meshes/v2/A_left_Degree4_link.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
- link A_left_Degree5_link: geometry collision mesh filename=package://bw_std_description/meshes/v2/A_left_Degree5_link.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; visual mesh filename=package://bw_std_description/meshes/v2/A_left_Degree5_link.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
- link A_left_Degree6_link: geometry collision mesh filename=package://bw_std_description/meshes/v2/A_left_Degree6_link.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; visual mesh filename=package://bw_std_description/meshes/v2/A_left_Degree6_link.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
- link A_left_Degree7_link: geometry collision mesh filename=package://bw_std_description/meshes/v2/A_left_Degree7_link.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; visual mesh filename=package://bw_std_description/meshes/v2/A_left_Degree7_link.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
- link A_left_Degree8_link: geometry collision mesh filename=package://bw_std_description/meshes/v2/A_left_Degree8_link.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; visual mesh filename=package://bw_std_description/meshes/v2/A_left_Degree8_link.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
- link A_left_Degree9_link: geometry collision mesh filename=package://bw_std_description/meshes/v2/A_left_Degree9_link.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; visual mesh filename=package://bw_std_description/meshes/v2/A_left_Degree9_link.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
- link A_right_Degree1_link: geometry collision mesh filename=package://bw_std_description/meshes/v2/A_right_Degree1_link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; visual mesh filename=package://bw_std_description/meshes/v2/A_right_Degree1_link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
- link A_right_Degree2_link: geometry collision mesh filename=package://bw_std_description/meshes/v2/A_right_Degree2_link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; visual mesh filename=package://bw_std_description/meshes/v2/A_right_Degree2_link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
- link A_right_Degree3_link: geometry collision mesh filename=package://bw_std_description/meshes/v2/A_right_Degree3_link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; visual mesh filename=package://bw_std_description/meshes/v2/A_right_Degree3_link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
- link A_right_Degree4_link: geometry collision mesh filename=package://bw_std_description/meshes/v2/A_right_Degree4_link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; visual mesh filename=package://bw_std_description/meshes/v2/A_right_Degree4_link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
- link A_right_Degree5_link: geometry collision mesh filename=package://bw_std_description/meshes/v2/A_right_Degree5_link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; visual mesh filename=package://bw_std_description/meshes/v2/A_right_Degree5_link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
- link A_right_Degree6_link: geometry collision mesh filename=package://bw_std_description/meshes/v2/A_right_Degree6_link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; visual mesh filename=package://bw_std_description/meshes/v2/A_right_Degree6_link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
- link A_right_Degree7_link: geometry collision mesh filename=package://bw_std_description/meshes/v2/A_right_Degree7_link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; visual mesh filename=package://bw_std_description/meshes/v2/A_right_Degree7_link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
- link A_right_Degree8_link: geometry collision mesh filename=package://bw_std_description/meshes/v2/A_right_Degree8_link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; visual mesh filename=package://bw_std_description/meshes/v2/A_right_Degree8_link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
- link A_right_Degree9_link: geometry collision mesh filename=package://bw_std_description/meshes/v2/A_right_Degree9_link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; visual mesh filename=package://bw_std_description/meshes/v2/A_right_Degree9_link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
- link C_Link: geometry collision mesh filename=package://bw_std_description/meshes/v2/C_Link.STL; visual mesh filename=package://bw_std_description/meshes/v2/C_Link.STL
Joints:
- removed joint D_behind_joint
- removed joint D_left_joint
- removed joint D_right_joint
- removed joint H_Degree1_joint
- removed joint H_Degree2_joint
- removed joint H_Degree3_joint
- removed joint base_footprint_to_base_link
- added joint chest_top_cap_joint: type fixed, parent C_Link, child chest_top_cap, origin xyz=0.092 0 0.0746 rpy=0 0 0
- added joint linear_slide_joint: type fixed, parent base_footprint, child linear_slide_link
- joint C_joint: parent base_link -> base_footprint

File: urdf/std_v3.urdf (robot description, URDF)
Before this commit: robot standard_patrol, 9 links, 8 joints
Links:
- link A_Degree1_Link: geometry collision mesh filename=package://bw_std_description/meshes/v3/A_Degree1_Link.STL; visual mesh filename=package://bw_std_description/meshes/v3/A_Degree1_Link.STL
- link A_Degree2_Link: geometry collision mesh filename=package://bw_std_description/meshes/v3/A_Degree2_Link.STL; visual mesh filename=package://bw_std_description/meshes/v3/A_Degree2_Link.STL
- link A_Degree3_Link: geometry collision mesh filename=package://bw_std_description/meshes/v3/A_Degree3_Link.STL; visual mesh filename=package://bw_std_description/meshes/v3/A_Degree3_Link.STL
- link C1_Link: geometry collision mesh filename=package://bw_std_description/meshes/v3/C1_Link.STL; visual mesh filename=package://bw_std_description/meshes/v3/C1_Link.STL
- link D_behind_Link: geometry collision mesh filename=package://bw_std_description/meshes/v3/D_behind_Link.STL; visual mesh filename=package://bw_std_description/meshes/v3/D_behind_Link.STL
- link D_left_Link: geometry collision mesh filename=package://bw_std_description/meshes/v3/D_left_Link.STL; visual mesh filename=package://bw_std_description/meshes/v3/D_left_Link.STL
- link D_right_Link: geometry collision mesh filename=package://bw_std_description/meshes/v3/D_right_Link.STL; visual mesh filename=package://bw_std_description/meshes/v3/D_right_Link.STL
- link base_link: geometry collision mesh filename=package://bw_std_description/meshes/v3/base_link.STL; visual mesh filename=package://bw_std_description/meshes/v3/base_link.STL

File: urdf/std_v4.urdf (robot description, URDF)
Before this commit: robot standard_arm, 14 links, 13 joints
Links:
- link A_right_Degree1_link: geometry collision mesh filename=package://bw_std_description/meshes/v4/A_right_Degree1_link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; visual mesh filename=package://bw_std_description/meshes/v4/A_right_Degree1_link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
- link A_right_Degree2_link: geometry collision mesh filename=package://bw_std_description/meshes/v4/A_right_Degree2_link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; visual mesh filename=package://bw_std_description/meshes/v4/A_right_Degree2_link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
- link A_right_Degree3_link: geometry collision mesh filename=package://bw_std_description/meshes/v4/A_right_Degree3_link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; visual mesh filename=package://bw_std_description/meshes/v4/A_right_Degree3_link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
- link A_right_Degree4_link: geometry collision mesh filename=package://bw_std_description/meshes/v4/A_right_Degree4_link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; visual mesh filename=package://bw_std_description/meshes/v4/A_right_Degree4_link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
- link A_right_Degree5_link: geometry collision mesh filename=package://bw_std_description/meshes/v4/A_right_Degree5_link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; visual mesh filename=package://bw_std_description/meshes/v4/A_right_Degree5_link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
- link A_right_Degree6_link: geometry collision mesh filename=package://bw_std_description/meshes/v4/A_right_Degree7_link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; visual mesh filename=package://bw_std_description/meshes/v4/A_right_Degree7_link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
- link A_right_Degree7_link: geometry collision mesh filename=package://bw_std_description/meshes/v4/A_right_Degree6_link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; visual mesh filename=package://bw_std_description/meshes/v4/A_right_Degree6_link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
- link A_right_Degree8_link: geometry collision mesh filename=package://bw_std_description/meshes/v4/A_right_Degree8_link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; visual mesh filename=package://bw_std_description/meshes/v4/A_right_Degree8_link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
- link A_right_Degree9_link: geometry collision mesh filename=package://bw_std_description/meshes/v4/A_right_Degree9_link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; visual mesh filename=package://bw_std_description/meshes/v4/A_right_Degree9_link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
- link D_behind_link: geometry collision mesh filename=package://bw_std_description/meshes/v4/D_behind_link.STL; visual mesh filename=package://bw_std_description/meshes/v4/D_behind_link.STL
- link D_left_link: geometry collision mesh filename=package://bw_std_description/meshes/v4/D_left_link.STL; visual mesh filename=package://bw_std_description/meshes/v4/D_left_link.STL
- link D_right_link: geometry collision mesh filename=package://bw_std_description/meshes/v4/D_right_link.STL; visual mesh filename=package://bw_std_description/meshes/v4/D_right_link.STL
- link base_link: geometry collision mesh filename=package://bw_std_description/meshes/v4/base_link.STL; visual mesh filename=package://bw_std_description/meshes/v4/base_link.STL
