Commit message: refactor(std): 扁平化描述包到仓库根目录并统一 std 命名
将 ROS 2 包从 src/standrad/ 扁平化到仓库根目录, 包名统一为 bw_std_description, 配套重命名 config、rviz、scripts、urdf 与 CMake 元数据。

运行时模型改名为 std_auto, 六个显示模型统一为 std_v1 至 std_v6, 生成脚本改为以 std_auto.urdf 为源模型输出显示模型。

启动参数 variant 改为 robot_model, 支持列表加入 std_auto, 非法取值直接报错并列出可选值, Gazebo 实体名默认改为 std_robot。

URDF 与 std_source.csv 中的资源引用统一为 package://bw_std_description/, Gazebo 启动时把该前缀替换为本地绝对路径。

117 个 STL 与 std.rviz、joint_names_std.yaml 仅移动或改名, 文件内容未变。

README 更新为新目录结构与新参数名, 补充 model、rviz_config、entity_name 等可选启动参数说明。

旧包名 standard 与旧参数 variant 不再支持。

File: urdf/std_v5.urdf (robot description, URDF)
Before this commit: robot standard_v5, 11 links, 10 joints
Links:
- link A_right_Degree1_link: geometry collision mesh filename=package://bw_std_description/meshes/v5/A_right_Degree1_link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; visual mesh filename=package://bw_std_description/meshes/v5/A_right_Degree1_link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
- link A_right_Degree2_link: geometry collision mesh filename=package://bw_std_description/meshes/v5/A_right_Degree2_link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; visual mesh filename=package://bw_std_description/meshes/v5/A_right_Degree2_link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
- link A_right_Degree3_link: geometry collision mesh filename=package://bw_std_description/meshes/v5/A_right_Degree3_link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; visual mesh filename=package://bw_std_description/meshes/v5/A_right_Degree3_link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
- link A_right_Degree4_link: geometry collision mesh filename=package://bw_std_description/meshes/v5/A_right_Degree4_link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; visual mesh filename=package://bw_std_description/meshes/v5/A_right_Degree4_link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
- link A_right_Degree5_link: geometry collision mesh filename=package://bw_std_description/meshes/v5/A_right_Degree5_link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; visual mesh filename=package://bw_std_description/meshes/v5/A_right_Degree5_link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
- link A_right_Degree6_link: geometry collision mesh filename=package://bw_std_description/meshes/v5/A_right_Degree7_link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; visual mesh filename=package://bw_std_description/meshes/v5/A_right_Degree7_link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
- link A_right_Degree7_link: geometry collision mesh filename=package://bw_std_description/meshes/v5/A_right_Degree6_link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; visual mesh filename=package://bw_std_description/meshes/v5/A_right_Degree6_link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
- link A_right_Degree8_link: geometry collision mesh filename=package://bw_std_description/meshes/v5/A_right_Degree8_link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; visual mesh filename=package://bw_std_description/meshes/v5/A_right_Degree8_link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
- link A_right_Degree9_link: geometry collision mesh filename=package://bw_std_description/meshes/v5/A_right_Degree9_link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; visual mesh filename=package://bw_std_description/meshes/v5/A_right_Degree9_link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
- link arm_base_plate_link: geometry collision mesh filename=package://bw_std_description/meshes/v5/v5_solid_base.STL; visual mesh filename=package://bw_std_description/meshes/v5/v5_solid_base.STL

File: urdf/std_v6.urdf (robot description, URDF)
Before this commit: robot standard_v6, 5 links, 4 joints
Links:
- link D_behind_link: geometry collision mesh filename=package://bw_std_description/meshes/v6/D_behind_link.STL; visual mesh filename=package://bw_std_description/meshes/v6/D_behind_link.STL
- link D_left_link: geometry collision mesh filename=package://bw_std_description/meshes/v6/D_left_link.STL; visual mesh filename=package://bw_std_description/meshes/v6/D_left_link.STL
- link D_right_link: geometry collision mesh filename=package://bw_std_description/meshes/v6/D_right_link.STL; visual mesh filename=package://bw_std_description/meshes/v6/D_right_link.STL
- link base_link: geometry collision mesh filename=package://bw_std_description/meshes/v6/v4_base_flat_top.STL; visual mesh filename=package://bw_std_description/meshes/v6/v4_base_flat_top.STL
